Commit message: Updated two arm setup

File: franka_description/robots/dual_panda_example.urdf.xacro (robot description, xacro)
@@ -8,7 +8,7 @@
   <link name="base">
     <visual>
-      <origin xyz="0 0 0.5" rpy="0 0 0"/>
+      <origin xyz="0 0 0.1" rpy="0 0 0"/>
       <geometry>
-        <box size="1 2 1" />
+        <box size="1 2 0.1" />
       </geometry>
       <material name="White">
@@ -17,15 +17,15 @@
     </visual>
     <collision>
-      <origin xyz="0 0 0.5" rpy="0 0 0"/>
+      <origin xyz="0 0 0.1" rpy="0 0 0"/>
       <geometry>
-        <box size="1 2 1" />
+        <box size="1 2 0.1" />
       </geometry>
     </collision>
   </link>
   <!-- right arm with gripper -->
-  <xacro:panda_arm arm_id="$(arg arm_id_1)" connected_to="base"  xyz="0 -0.5 1" />
+  <xacro:panda_arm arm_id="$(arg arm_id_1)" connected_to="base"  xyz="0 0.0 0.1" />
   <xacro:hand ns="$(arg arm_id_1)" rpy="0 0 ${-pi/4}" connected_to="$(arg arm_id_1)_link8" />
   <!-- left arm with gripper -->
-  <xacro:panda_arm arm_id="$(arg arm_id_2)" connected_to="base"  xyz="0 0.5 1" />
+  <xacro:panda_arm arm_id="$(arg arm_id_2)" connected_to="base"  xyz="0.015 -0.660 0.1" />
   <xacro:hand ns="$(arg arm_id_2)" rpy="0 0 ${-pi/4}" connected_to="$(arg arm_id_2)_link8" />
 </robot>

Commit message: Update urdf

File: franka_description/robots/dual_panda_example.urdf.xacro (robot description, xacro)
@@ -8,5 +8,5 @@
   <link name="base">
     <visual>
-      <origin xyz="0 0 0.1" rpy="0 0 0"/>
+      <origin xyz="0 0 0.0" rpy="0 0 0"/>
       <geometry>
         <box size="1 2 0.1" />
@@ -17,5 +17,5 @@
     </visual>
     <collision>
-      <origin xyz="0 0 0.1" rpy="0 0 0"/>
+      <origin xyz="0 0 0.0" rpy="0 0 0"/>
       <geometry>
         <box size="1 2 0.1" />
@@ -24,8 +24,8 @@
   </link>
   <!-- right arm with gripper -->
-  <xacro:panda_arm arm_id="$(arg arm_id_1)" connected_to="base"  xyz="0 0.0 0.1" />
+  <xacro:panda_arm arm_id="$(arg arm_id_1)" connected_to="base"  xyz="0 0.0 0.0" />
   <xacro:hand ns="$(arg arm_id_1)" rpy="0 0 ${-pi/4}" connected_to="$(arg arm_id_1)_link8" />
   <!-- left arm with gripper -->
-  <xacro:panda_arm arm_id="$(arg arm_id_2)" connected_to="base"  xyz="-0.015 0.660 0.1" />
+  <xacro:panda_arm arm_id="$(arg arm_id_2)" connected_to="base"  xyz="-0.015 0.660 0.0" />
   <xacro:hand ns="$(arg arm_id_2)" rpy="0 0 ${-pi/4}" connected_to="$(arg arm_id_2)_link8" />
 </robot>

Commit message: Update urdf

File: franka_description/robots/dual_panda_example.urdf.xacro (robot description, xacro)
@@ -16,10 +16,10 @@
       </material>
     </visual>
-    <collision>
-      <origin xyz="0 0 0.0" rpy="0 0 0"/>
-      <geometry>
-        <box size="1 2 0.1" />
-      </geometry>
-    </collision>
+    <!-- <collision> -->
+      <!-- <origin xyz="0 0 0.0" rpy="0 0 0"/> -->
+      <!-- <geometry> -->
+        <!-- <box size="1 2 0.1" /> -->
+      <!-- </geometry> -->
+    <!-- </collision> -->
   </link>
   <!-- right arm with gripper -->

Commit message: Update urdf

File: franka_description/robots/dual_panda_example.urdf.xacro (robot description, xacro)
@@ -17,9 +17,9 @@
     </visual>
     <!-- <collision> -->
-      <!-- <origin xyz="0 0 0.0" rpy="0 0 0"/> -->
-      <!-- <geometry> -->
-        <!-- <box size="1 2 0.1" /> -->
-      <!-- </geometry> -->
-    <!-- </collision> -->
+      <origin xyz="0 0 0.0" rpy="0 0 0"/>
+      <geometry>
+        <box size="0 0 0" />
+      </geometry>
+    </collision>
   </link>
   <!-- right arm with gripper -->

Commit message: Update urdf

File: franka_description/robots/dual_panda_example.urdf.xacro (robot description, xacro)
@@ -16,5 +16,5 @@
       </material>
     </visual>
-    <!-- <collision> -->
+    <collision>
       <origin xyz="0 0 0.0" rpy="0 0 0"/>
       <geometry>
