Commit message: Updated joint limit for joint 7

File: franka_description/robots/panda_arm.xacro (robot description, xacro)
@@ -278,10 +278,11 @@
     </link>
     <joint name="${arm_id}_joint7" type="revolute">
-      <safety_controller k_position="100.0" k_velocity="40.0" soft_lower_limit="-2.8973" soft_upper_limit="2.8973"/>
+      <!-- <safety_controller k_position="100.0" k_velocity="40.0" soft_lower_limit="-2.8973" soft_upper_limit="2.8973"/> -->
+      <safety_controller k_position="100.0" k_velocity="40.0" soft_lower_limit="-2.8" soft_upper_limit="1.64"/>
       <origin rpy="${pi/2} 0 0" xyz="0.088 0 0"/>
       <parent link="${arm_id}_link6"/>
       <child link="${arm_id}_link7"/>
       <axis xyz="0 0 1"/>
-      <limit effort="12" lower="-2.8973" upper="2.8973" velocity="2.6100"/>
+      <limit effort="12" lower="-2.8" upper="1.64" velocity="2.6100"/>
     </joint>
     <link name="${arm_id}_link8">

Commit message: Modified joint limits

File: franka_description/robots/panda_arm.xacro (robot description, xacro)
@@ -62,10 +62,12 @@
     </link>
     <joint name="${arm_id}_joint1" type="revolute">
-      <safety_controller k_position="100.0" k_velocity="40.0" soft_lower_limit="-2.8973" soft_upper_limit="2.8973"/>
+      <!-- <safety_controller k_position="100.0" k_velocity="40.0" soft_lower_limit="-2.8973" soft_upper_limit="2.8973"/> -->
+      <safety_controller k_position="100.0" k_velocity="40.0" soft_lower_limit="-2.85" soft_upper_limit="2.85"/>
       <origin rpy="0 0 0" xyz="0 0 0.333"/>
       <parent link="${arm_id}_link0"/>
       <child link="${arm_id}_link1"/>
       <axis xyz="0 0 1"/>
-      <limit effort="87" lower="-2.8973" upper="2.8973" velocity="2.1750"/>
+      <!-- <limit effort="87" lower="-2.8973" upper="2.8973" velocity="2.1750"/> -->
+      <limit effort="87" lower="-2.85" upper="2.85" velocity="2.1750"/>
     </joint>
     <link name="${arm_id}_link2">
@@ -128,10 +130,11 @@
     </link>
     <joint name="${arm_id}_joint3" type="revolute">
-      <safety_controller k_position="100.0" k_velocity="40.0" soft_lower_limit="-2.8973" soft_upper_limit="2.8973"/>
+      <!-- <safety_controller k_position="100.0" k_velocity="40.0" soft_lower_limit="-2.8973" soft_upper_limit="2.8973"/> -->
+      <safety_controller k_position="100.0" k_velocity="40.0" soft_lower_limit="-2.85" soft_upper_limit="2.85"/>
       <origin rpy="${pi/2} 0 0" xyz="0 -0.316 0"/>
       <parent link="${arm_id}_link2"/>
       <child link="${arm_id}_link3"/>
       <axis xyz="0 0 1"/>
-      <limit effort="87" lower="-2.8973" upper="2.8973" velocity="2.1750"/>
+      <limit effort="87" lower="-2.85" upper="2.85" velocity="2.1750"/>
     </joint>
     <link name="${arm_id}_link4">
@@ -161,10 +164,12 @@
     </link>
     <joint name="${arm_id}_joint4" type="revolute">
-      <safety_controller k_position="100.0" k_velocity="40.0" soft_lower_limit="-3.0718" soft_upper_limit="-0.0698"/>
+      <!-- <safety_controller k_position="100.0" k_velocity="40.0" soft_lower_limit="-3.0718" soft_upper_limit="-0.0698"/> -->
+      <safety_controller k_position="100.0" k_velocity="40.0" soft_lower_limit="-2.7" soft_upper_limit="-0.10"/>
       <origin rpy="${pi/2} 0 0" xyz="0.0825 0 0"/>
       <parent link="${arm_id}_link3"/>
       <child link="${arm_id}_link4"/>
       <axis xyz="0 0 1"/>
-      <limit effort="87" lower="-3.0718" upper="-0.0698" velocity="2.1750"/>
+      <!-- <limit effort="87" lower="-3.0718" upper="-0.0698" velocity="2.1750"/> -->
+      <limit effort="87" lower="-2.7" upper="-0.10" velocity="2.1750"/>
     </joint>
     <link name="${arm_id}_link5">
@@ -212,10 +217,12 @@
     </link>
     <joint name="${arm_id}_joint5" type="revolute">
-      <safety_controller k_position="100.0" k_velocity="40.0" soft_lower_limit="-2.8973" soft_upper_limit="2.8973"/>
+      <!-- <safety_controller k_position="100.0" k_velocity="40.0" soft_lower_limit="-2.8973" soft_upper_limit="2.8973"/> -->
+      <safety_controller k_position="100.0" k_velocity="40.0" soft_lower_limit="-2.85" soft_upper_limit="2.85"/>
       <origin rpy="${-pi/2} 0 0" xyz="-0.0825 0.384 0"/>
       <parent link="${arm_id}_link4"/>
       <child link="${arm_id}_link5"/>
       <axis xyz="0 0 1"/>
-      <limit effort="12" lower="-2.8973" upper="2.8973" velocity="2.6100"/>
+      <!-- <limit effort="12" lower="-2.8973" upper="2.8973" velocity="2.6100"/> -->
+      <limit effort="12" lower="-2.85" upper="2.85" velocity="2.6100"/>
     </joint>
     <link name="${arm_id}_link6">
@@ -245,10 +252,12 @@
     </link>
     <joint name="${arm_id}_joint6" type="revolute">
-      <safety_controller k_position="100.0" k_velocity="40.0" soft_lower_limit="-0.0175" soft_upper_limit="3.7525"/>
+      <!-- <safety_controller k_position="100.0" k_velocity="40.0" soft_lower_limit="-0.0175" soft_upper_limit="3.7525"/> -->
+      <safety_controller k_position="100.0" k_velocity="40.0" soft_lower_limit="0.3" soft_upper_limit="3.7"/>
       <origin rpy="${pi/2} 0 0" xyz="0 0 0"/>
       <parent link="${arm_id}_link5"/>
       <child link="${arm_id}_link6"/>
       <axis xyz="0 0 1"/>
-      <limit effort="12" lower="-0.0175" upper="3.7525" velocity="2.6100"/>
+      <!-- <limit effort="12" lower="-0.0175" upper="3.7525" velocity="2.6100"/> -->
+      <limit effort="12" lower="0.3" upper="3.7" velocity="2.6100"/>
     </joint>
     <link name="${arm_id}_link7">
@@ -279,10 +288,11 @@
     <joint name="${arm_id}_joint7" type="revolute">
       <!-- <safety_controller k_position="100.0" k_velocity="40.0" soft_lower_limit="-2.8973" soft_upper_limit="2.8973"/> -->
-      <safety_controller k_position="100.0" k_velocity="40.0" soft_lower_limit="-2.8" soft_upper_limit="1.64"/>
+      <safety_controller k_position="100.0" k_velocity="40.0" soft_lower_limit="-2.7" soft_upper_limit="2.7"/>
       <origin rpy="${pi/2} 0 0" xyz="0.088 0 0"/>
       <parent link="${arm_id}_link6"/>
       <child link="${arm_id}_link7"/>
       <axis xyz="0 0 1"/>
-      <limit effort="12" lower="-2.8" upper="1.64" velocity="2.6100"/>
+      <!-- <limit effort="12" lower="-2.8973" upper="2.8973" velocity="2.6100"/> -->
+      <limit effort="12" lower="-2.7" upper="2.7" velocity="2.6100"/>
     </joint>
     <link name="${arm_id}_link8">
